File: PCB/right/right.kicad_pcb (KiCad board)
At the start: 2 copper layers, 130 x 109 mm, 49 parts, among them SW1 SW_Push_45deg, SW10 SW_Push_45deg, SW11 SW_Push_45deg, SW12 SW_Push_45deg, SW13 SW_Push_45deg, SW14 SW_Push_45deg, SW15 SW_Push_45deg, SW16 SW_Push_45deg, SW17 SW_Push_45deg, SW18 SW_Push_45deg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

Commit message: [ JUN 21 // MODEL ]
Connections:
- A1 pad 39: unconnected-(A1-VSYS-Pad39) -> Net-(A1-VSYS)
- A1 pad 40: Net-(A1-VBUS) -> unconnected-(A1-VBUS-Pad40)
- U2 pad 2: Net-(A1-VBUS) -> Net-(A1-VSYS)
Routing:
- net Net-(A1-VBUS): track 97.1 -> 0.00 mm, vias 2 -> 0
- net Net-(A1-VSYS): track 0.00 -> 96.4 mm, vias 0 -> 2
