File: PCB/right/right.kicad_sch (KiCad schematic)
At the start: 49 parts, among them SW1 SW_Push_45deg, SW10 SW_Push_45deg, SW11 SW_Push_45deg, SW12 SW_Push_45deg, SW13 SW_Push_45deg, SW14 SW_Push_45deg, SW15 SW_Push_45deg, SW16 SW_Push_45deg, SW17 SW_Push_45deg, SW18 SW_Push_45deg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

Commit message: [ JUN 21 // MODEL ]
Connections:
- net at A1.39 (VSYS): now also U2.2 (TIP)
- net at A1.40 (VBUS): no longer U2.2 (TIP)
- no-connect marks 17 -> 16
Changed lines of the file:
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@@
-	)
-	(no_connect
-		(at 58.42 29.21)
 	)
 	(no_connect
@@
 	(wire
 		(pts
+			(xy 58.42 15.24) (xy 58.42 29.21)
+		)
+		(stroke
+			(width 0)
+			(type default)
+		)
+	)
+	(wire
+		(pts
 			(xy 205.74 29.21) (xy 205.74 40.64)
 		)
@@
 	(wire
 		(pts
+			(xy 58.42 15.24) (xy 123.19 15.24)
+		)
+		(stroke
+			(width 0)
+			(type default)
+		)
+	)
+	(wire
+		(pts
 			(xy 40.64 142.24) (xy 48.26 142.24)
 		)
@@
 	(wire
 		(pts
-			(xy 63.5 29.21) (xy 63.5 15.24)
-		)
-		(stroke
-			(width 0)
-			(type default)
-		)
-	)
-	(wire
-		(pts
 			(xy 73.66 175.26) (xy 105.41 175.26)
 		)
@@
 		)
 		(stroke
-			(width 0)
-			(type default)
-		)
-	)
-	(wire
-		(pts
-			(xy 63.5 15.24) (xy 123.19 15.24)
-		)
-		(stroke
